File: Untitled.kicad_sch (KiCad schematic)
At the start: 2 parts

Commit message: changed text
Other:
- note added: "THIS IS THE SECOND CHANGE TEST"
Changed lines of the file:
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@@
 (kicad_sch (version 20230121) (generator eeschema)
   (paper "A4")
+  (text "THIS IS THE SECOND CHANGE TEST" (at 80.645 106.045 0)
+    (effects (font (size 1.27 1.27)) (justify left bottom))
+  )
   (symbol (lib_id "Device:R_Photo") (at 124.46 74.93 0) (unit 1)
     (in_bom yes) (on_board yes) (dnp no) (fields_autoplaced)

Commit message: done with 1st draft schematic
done with 1st draft schematic
Parts:
- removed R1: R_Photo, symbol Device:R_Photo
- removed TH1: Thermistor_PTC_3Wire, symbol Device:Thermistor_PTC_3Wire
- added BT1: 3v, symbol Device:Battery
- added C1: 5pF, symbol Device:C_Small
- added C2: 2.7nF, symbol Device:C_Small
- added C3, C4, C5: 10uF, symbol Device:C_Small
- added C6: 1uF, symbol Device:C_Small
- added C7, C8: 0.1uF, symbol Device:C_Small
- added D1: LED, symbol Device:LED
- added IC_Reg: LP38511MRX REGULATOR, MRA08B, symbol 2023-10-17_22-37-01:LP38511MRX-ADJ_NOPB
- added R1: 20k, symbol Device:R_Small
- added R2: 2k, symbol Device:R_Small
- added R3: 357, symbol Device:R_Small
- added R4, R5: 10k, symbol Device:R_Small
- added R6: 52, symbol Device:R_Small
- added SW1: SW_Push, symbol Switch:SW_Push
- added U1: ESP32-C3-MINI-1-N4, ESP32-C3-MINI-1_EXP, symbol 2023-10-17_22-30-38:ESP32-C3-MINI-1-N4
- added U2: ~, symbol Library for HOPE PROJECT:Haptic_Motor
- added U3: Opamp_Dual, symbol Device:Opamp_Dual
- added U4: ~, symbol Library for HOPE PROJECT:Photodiode_SD019-141-411-X
Connections:
- new net: C2.2, IC_Reg.3 (ADJ), R2.2, R3.1
- new net: D1.2 (A), R6.2
- new net 3v3: C2.1, C4.1, C5.1, C7.1, IC_Reg.1 (OUT), IC_Reg.2 (OUT), R2.1, R4.1, R5.1, U1.3 (3V3)
- new net GND: BT1.2 (-), C3.2, C4.2, C5.2, C6.2, C7.2, C8.2, D1.1 (K), IC_Reg.5 (GND), R3.2, SW1.1, U1.1 (GND), U1.11 (GND), U1.2 (GND), U1.36 (GND), U1.37 (GND), U1.38 (GND), U1.39 (GND), U1.40 (GND), U1.41 (GND), U1.42 (GND), U1.43 (GND), U1.44 (GND), U1.45 (GND), U1.46 (GND), U1.47 (GND), U1.48 (GND), U1.49 (GND), U1.50 (GND), U1.51 (GND), U1.52 (GND), U1.53 (GND), U1.54 (GND), U1.55 (GND), U1.56 (GND), U1.57 (GND), U1.58 (GND), U1.59 (GND), U1.60 (GND), U1.61 (GND), U2.1 (GND), U3.3 (+), U3.4 (V-), U4.1 (+)
- new net IO2: R5.2, U1.5 (IO2)
- new net LED_in: R6.1, U1.23 (IO9)
- new net Photo_Out: C1.1, R1.2, U1.26 (IO18), U3.1
- new net Photodiode Input: C1.2, R1.1, U3.2 (-), U4.2 (-)
- new net Vdd: BT1.1 (+), C3.1, IC_Reg.7 (IN), IC_Reg.8 (IN), U3.8 (V+)
- new net en: C6.1, C8.1, IC_Reg.6 (EN), R4.2, SW1.2, U1.8 (EN)
- new net haptic_input_Vin: U1.13 (IO1), U2.0 (Vin)
Other:
- note added: "0.1mA IN"
- note added: "3.3v"
- note added: "3.3v IN"
- note added: "3.3v OUT"
- note added: "3v"
- note added: "< 2v IN"
- note added: "ESP32"
- note added: "Regulator"
- note added: "output of sensor < 2v"
- note added: "~0.1mA"
- note added: "~0.1mA OUT"
- note added: "~20mA forward current"
- note removed: "THIS IS THE SECOND CHANGE TEST"
